File: Hardware/Basic/Bottom/SmartWatch-BASIC-Bottom.brd (EAGLE design)
At the start: 33 x 33 mm, 31 parts, among them U1 AD5242-SO16

Commit message: take 2
Parts:
- added J1: (no value), LinnesLab-Connectors:1X07
- moved C21 38.7 mm to (7.62, 7.62)
- moved R24 33.5 mm to (12.7, 14.0)
- moved C20 32.1 mm to (12.7, 22.9)
- moved R20 31.4 mm to (6.35, 26.7)
- moved C22 31.1 mm to (12.7, 11.4)
- moved R21 30.9 mm to (6.35, 22.9)
- moved R22 30.9 mm to (6.35, 17.8)
- moved C19 30.5 mm to (6.35, 14.0)
- moved OP4 29.0 mm to (17.8, 26.7)
- moved R23 28.7 mm to (7.62, 11.4)
- moved R19 16.1 mm to (30.5, 27.9)
- moved C10 10.9 mm to (28.7, 31.6)
- moved C15 9.25 mm to (22.3, 32.3)
- moved C11 9.16 mm to (12.2, 26.5)
- moved R13 8.13 mm to (12.2, 29.3)
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Connections:
- removed net LED.CTRL: U$4.8
- removed net PPG: C21.2, OP3.1, U1.14
- removed net TIA: C10.2, C15.1, OP4.1, U1.3
- new net A6/TIA: C10.2, C15.1, J1.5, OP4.1, U1.3
- new net A7/PPG: C21.2, J1.7, OP3.1, U1.14
- new net D29/LED.CTRL: J1.6, U$4.8
- new net N$7: J1.1
- net 3.3V: now also J1.3
- net GND: now also J1.2
- net SCL: now also J1.4

Commit message: take3
Parts:
- moved R17 53.2 mm to (45.0, -5.57)
- moved R21 50.7 mm to (42.3, -12.9), turned to 180 degrees
- moved R18 49.8 mm to (45.0, -4.28), turned to 180 degrees
- moved R22 47.2 mm to (44.5, -9.96), turned to 270 degrees
- moved C16 47.2 mm to (38.9, -14.8)
- moved C19 47.0 mm to (46.8, -9.96), turned to 90 degrees
- moved R23 46.9 mm to (49.3, -10.0), turned to 90 degrees
- moved R20 46.2 mm to (25.2, -15.5)
- moved R15 44.3 mm to (38.8, -12.9), turned to 180 degrees
- moved C14 43.4 mm to (21.3, -12.4)
- moved R13 42.9 mm to (30.9, -9.41)
- moved R14 42.9 mm to (26.9, -11.4)
- moved R19 40.5 mm to (31.4, -12.5)
- moved C15 40.0 mm to (29.4, -7.06), turned to 0 degrees
- moved C11 39.8 mm to (33.5, -7.12), turned to 270 degrees
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Connections:
- removed net LED: Q1.3
- net LED.C: now also Q1.3
Routing:
- net N$19: track 0.00 -> 22.7 mm
- net N$18: track 0.00 -> 7.54 mm
- net N$17: track 0.00 -> 3.63 mm
- net N$10: track 0.00 -> 2.92 mm
- net GND: track 0.00 -> 2.88 mm, vias 0 -> 2
- net G.W2: track 0.00 -> 2.19 mm
- net A7/PPG: track 0.00 -> 2.19 mm
- net VREF: track 0.00 -> 1.27 mm
- added copper zone on layer 16, net GND

Commit message: take3_1_24
Parts:
- removed OP4: (no value), LinnesLab-AnalogIC:SOT23-5
- removed U$4: AD5171, LinnesLab-DigitalIC:SOT-23-8
- removed U1: AD5242-SO16, LinnesLab-DigitalIC:SO16
- added AD5171: AD5171, LinnesLab-DigitalIC:SOT-23-8
- added AD5242: AD5242-SO16, LinnesLab-DigitalIC:SO16
- added TIA: (no value), LinnesLab-AnalogIC:SOT23-5
- J1: device LinnesLab-Connectors:1X07 -> LinnesLab-Connectors:1X07_1.27MM
- moved R23 41.5 mm to (28.8, 26.1), turned to 180 degrees
- moved C19 38.1 mm to (28.8, 23.6), turned to 180 degrees
- moved R22 35.1 mm to (28.8, 21.3), turned to 0 degrees
- moved R17 34.2 mm to (24.5, 21.8), turned to 90 degrees
- moved R18 33.9 mm to (23.4, 21.8), turned to 270 degrees
- moved R21 33.7 mm to (31.7, 19.1), turned to 270 degrees
- moved C16 30.7 mm to (33.6, 15.5), turned to 90 degrees
- moved R15 29.3 mm to (32.1, 15.6), turned to 270 degrees
- moved OP3 26.8 mm to (25.6, 16.2), turned to 0 degrees
- moved C18 24.6 mm to (5.56, 9.54), turned to 270 degrees
- moved R19 23.6 mm to (33.0, 11.0), turned to 270 degrees
- moved C22 22.9 mm to (14.1, 22.0)
- moved C14 22.6 mm to (30.0, 8.53), turned to 180 degrees
- moved R20 22.6 mm to (29.9, 6.60), turned to 180 degrees
- moved R14 22.2 mm to (29.9, 10.6), turned to 0 degrees
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Connections:
- removed net N$7: J1.1
- net 3.3V: now also AD5171.2, AD5171.6, AD5242.5, AD5242.6, J1.4, TIA.5; no longer J1.3, OP4.5, U$4.2, U$4.6, U1.5, U1.6
- net A6/TIA: now also AD5242.3, J1.6, TIA.1; no longer J1.5, OP4.1, U1.3
- net A7/PPG: now also AD5242.14; no longer U1.14
- net D29/LED.CTRL: now also AD5171.8, J1.5; no longer J1.6, U$4.8
- net G.A1: now also AD5242.2; no longer U1.2
- net G.A2: now also AD5242.16; no longer U1.16
- net G.O1: now also AD5242.1; no longer U1.1
- net G.O2: now also AD5242.13; no longer U1.13
- net G.W2: now also AD5242.15; no longer U1.15
- net GND: now also AD5171.3, AD5242.10, AD5242.11, AD5242.12, AD5242.9, J1.3, TIA.2, TIA.3; no longer J1.2, OP4.2, OP4.3, U$4.3, U1.10, U1.11, U1.12, U1.9
- net N$9: now also AD5171.1, AD5171.7; no longer U$4.1, U$4.7
- net PD.C: now also AD5242.4, TIA.4; no longer OP4.4, U1.4
- net SCL: now also AD5171.4, AD5242.7, J1.2; no longer J1.4, U$4.4, U1.7
- net SDA: now also AD5171.5, AD5242.8, J1.1; no longer U$4.5, U1.8
Routing:
- net A6/TIA: track 0.00 -> 68.9 mm, vias 0 -> 4
- net A7/PPG: track 2.19 -> 50.1 mm
- net VREF: track 1.27 -> 35.3 mm, vias 0 -> 3
- net SDA: track 0.00 -> 33.7 mm
- net SCL: track 0.00 -> 33.2 mm, vias 0 -> 2
- net GND: track 2.88 -> 28.9 mm, vias 2 -> 15
- net PD.C: track 0.00 -> 23.4 mm, vias 0 -> 2
- net N$9: track 0.00 -> 21.3 mm
- net N$13: track 0.00 -> 18.3 mm
- net D29/LED.CTRL: track 0.00 -> 17.2 mm, vias 0 -> 2
- net G.W2: track 2.19 -> 16.0 mm, vias 0 -> 2
- net N$16: track 0.00 -> 10.3 mm
- net N$15: track 0.00 -> 7.40 mm
- net N$17: track 3.63 -> 9.95 mm, vias 0 -> 2
- net N$20: track 0.00 -> 2.36 mm
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
Commit message: Take5
Parts:
- added C1: 100n, LinnesLab-Passives:C0603
- added LOGO1: REVISION.A, LinnesLab-Logos:REV.A
- moved OP3 0.39 mm to (26.0, 16.3)
- moved C21 0.20 mm to (22.6, 11.4)
Connections:
- net GND: now also C1.1
- net VREF: now also C1.2
Routing:
- net GND: track 28.9 -> 30.5 mm, vias 15 -> 16
- net N$19: track 21.6 -> 22.7 mm
- net N$17: track 9.95 -> 10.9 mm
- net N$10: track 2.87 -> 3.50 mm

Commit message: take6
Parts:
- added C2, C7, C9: 1u, LinnesLab-Passives:C0603
- added C3, C5: 4.7u, LinnesLab-Passives:C0603
- added CHRG1: MCP73831, LinnesLab-Power:SOT23-5
- added LDO1: MIC5504, LinnesLab-Power:SOT23-5
- added R3: 100k, LinnesLab-Passives:R0603
- added R5: (no value), LinnesLab-Passives:R0603
- added U3: PCF8523, LinnesLab-Clocks:SO8
- added XTAL2: 32.7680kHz, LinnesLab-Clocks:2-SMD.NOLEAD.2.0MMTO1.2MM
Connections:
- new net D27/CHRG.STATUS: CHRG1.1, R3.1
- new net N$2: U3.2, XTAL2.P$1
- new net N$3: U3.1, XTAL2.P$2
- new net N$4: CHRG1.5, R5.2
- new net VBATT: U3.3
- new net VIN1: C5.2, C7.2, CHRG1.4, LDO1.1, LDO1.3, R3.2
- new net VLIPO: C3.1, CHRG1.3
- net 3.3V: now also C2.1, C9.1, LDO1.5, U3.8
- net GND: now also C2.2, C3.2, C5.1, C7.1, C9.2, CHRG1.2, LDO1.2, R5.1, U3.4
- net SCL: now also U3.6
- net SDA: now also U3.5

Commit message: 'take8'
Parts:
- removed C3, C5: 4.7u, LinnesLab-Passives:C0603
- removed C7, C9: 1u, LinnesLab-Passives:C0603
- removed CHRG1: MCP73831, LinnesLab-Power:SOT23-5
- removed LDO1: MIC5504, LinnesLab-Power:SOT23-5
- removed R3: 100k, LinnesLab-Passives:R0603
- removed R5: (no value), LinnesLab-Passives:R0603
- moved C2 52.9 mm to (33.5, 31.8), turned to 270 degrees
- moved XTAL2 51.6 mm to (24.7, 32.4), turned to 90 degrees
- moved U3 48.5 mm to (29.4, 31.4)
- moved C15 4.01 mm to (26.3, 5.25)
- moved C1 3.02 mm to (30.6, 27.7), turned to 180 degrees
- moved LOGO1 2.45 mm to (31.5, 34.5)
- moved R14 0.74 mm to (29.1, 10.5)
- moved R13 0.69 mm to (32.7, 6.75)
- moved C14 0.69 mm to (29.3, 8.63)
- moved R20 0.61 mm to (29.3, 6.55)
- moved C16 0.31 mm to (33.3, 15.6)
- moved R15 0.18 mm to (31.9, 15.6)
Connections:
- net A6/TIA renamed A5/TIA
- net A7/PPG renamed A4/PPG
- net D29/LED.CTRL renamed D30/LED.CTRL
- removed net D27/CHRG.STATUS: CHRG1.1, R3.1
- removed net N$4: CHRG1.5, R5.2
- removed net VIN1: C5.2, C7.2, CHRG1.4, LDO1.1, LDO1.3, R3.2
- removed net VLIPO: C3.1, CHRG1.3
- net 3.3V: no longer C9.1, LDO1.5
- net GND: no longer C3.2, C5.1, C7.1, C9.2, CHRG1.2, LDO1.2, R5.1
Routing:
- net SDA: track 33.7 -> 62.0 mm, vias 0 -> 2
- net SCL: track 33.2 -> 59.9 mm, vias 2 -> 4
- net A5/TIA: track 68.6 -> 63.6 mm
- net GND: track 30.5 -> 34.0 mm, vias 16 -> 18
- net N$2: track 0.00 -> 2.22 mm
- net N$3: track 0.00 -> 2.09 mm
- net N$13: track 18.7 -> 17.8 mm
- net N$9: track 21.3 -> 22.0 mm, vias 0 -> 2
- net D30/LED.CTRL: track 17.2 -> 17.3 mm, vias 2 -> 4
