File: Hardware/Basic/Bottom/SmartWatch-BASIC-Bottom.sch (EAGLE design)
At the start: 31 parts, among them U1 AD5242-SO16

Commit message: take 2
Parts:
- added J1: (no value), LinnesLab-Connectors:CONN_07
Connections:
- removed net LED.CTRL: U$4.A
- removed net PPG: C21.2, OP3G$1.OUT, U1.B2
- removed net TIA: C10.2, C15.1, OP4G$1.OUT, U1.W1
- new net A6/TIA: C10.2, C15.1, J1.5, OP4G$1.OUT, U1.W1
- new net A7/PPG: C21.2, J1.7, OP3G$1.OUT, U1.B2
- new net D29/LED.CTRL: J1.6, U$4.A
- new net N$7: J1.1
- net 3.3V: now also J1.3
- net GND: now also J1.2
- net SCL: now also J1.4
Changed lines of the file:
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@@
 <part name="GND32" library="LinnesLab-Symbols" deviceset="GND" device=""/>
 <part name="SUPPLY26" library="LinnesLab-Symbols" deviceset="3.3V" device=""/>
+<part name="J1" library="LinnesLab-Connectors" deviceset="CONN_07" device=""/>
 </parts>
 <sheets>
@@
 <attribute name="VALUE" x="10.16" y="2.794" size="1.778" layer="96" align="bottom-center"/>
 </instance>
+<instance part="J1" gate="G$1" x="93.98" y="-12.7" smashed="yes">
+<attribute name="VALUE" x="88.9" y="-22.606" size="1.778" layer="96" font="vector"/>
+<attribute name="NAME" x="88.9" y="0.508" size="1.778" layer="95" font="vector"/>
+</instance>
 </instances>
 <busses>
@@
 <wire x1="10.16" y1="-12.7" x2="10.16" y2="-10.16" width="0.1524" layer="91"/>
 </segment>
+<segment>
+<pinref part="J1" gate="G$1" pin="2"/>
+<wire x1="99.06" y1="-15.24" x2="104.14" y2="-15.24" width="0.1524" layer="91"/>
+<label x="104.14" y="-15.24" size="1.016" layer="95" xref="yes"/>
+</segment>
 </net>
 <net name="3.3V" class="0">
@@
 <wire x1="10.16" y1="0" x2="10.16" y2="-2.54" width="0.1524" layer="91"/>
 </segment>
+<segment>
+<pinref part="J1" gate="G$1" pin="3"/>
+<wire x1="99.06" y1="-12.7" x2="104.14" y2="-12.7" width="0.1524" layer="91"/>
+<label x="104.14" y="-12.7" size="1.016" layer="95" xref="yes"/>
+</segment>
 </net>
 <net name="SDA" class="0">
@@
 <label x="50.8" y="-10.16" size="1.27" layer="95" xref="yes"/>
 </segment>
-</net>
-<net name="TIA" class="0">
+<segment>
+<pinref part="J1" gate="G$1" pin="4"/>
+<wire x1="99.06" y1="-10.16" x2="104.14" y2="-10.16" width="0.1524" layer="91"/>
+<label x="104.14" y="-10.16" size="1.016" layer="95" xref="yes"/>
+</segment>
+</net>
+<net name="A6/TIA" class="0">
 <segment>
 <wire x1="119.38" y1="33.02" x2="114.3" y2="33.02" width="0.1524" layer="91"/>
@@
 <junction x="66.04" y="99.06"/>
 </segment>
+<segment>
+<pinref part="J1" gate="G$1" pin="5"/>
+<wire x1="99.06" y1="-7.62" x2="104.14" y2="-7.62" width="0.1524" layer="91"/>
+<label x="104.14" y="-7.62" size="1.016" layer="95" xref="yes"/>
+</segment>
 </net>
 <net name="PD.C" class="0">
@@
 </segment>
 </net>
-<net name="LED.CTRL" class="0">
+<net name="D29/LED.CTRL" class="0">
 <segment>
 <pinref part="U$4" gate="G$1" pin="A"/>
@@
 <wire x1="215.9" y1="35.56" x2="215.9" y2="43.18" width="0.1524" layer="91"/>
 <label x="215.9" y="43.18" size="1.27" layer="95" rot="R180" xref="yes"/>
+</segment>
+<segment>
+<pinref part="J1" gate="G$1" pin="6"/>
+<wire x1="99.06" y1="-5.08" x2="104.14" y2="-5.08" width="0.1524" layer="91"/>
+<label x="104.14" y="-5.08" size="1.016" layer="95" xref="yes"/>
 </segment>
 </net>
@@
 </segment>
 </net>
-<net name="PPG" class="0">
+<net name="A7/PPG" class="0">
 <segment>
 <wire x1="147.32" y1="33.02" x2="149.86" y2="33.02" width="0.1524" layer="91"/>
@@
 <label x="205.74" y="111.76" size="1.27" layer="95" rot="R180" xref="yes"/>
 <label x="205.74" y="91.44" size="1.27" layer="95" xref="yes"/>
+</segment>
+<segment>
+<pinref part="J1" gate="G$1" pin="7"/>
+<wire x1="99.06" y1="-2.54" x2="104.14" y2="-2.54" width="0.1524" layer="91"/>
+<label x="104.14" y="-2.54" size="1.016" layer="95" xref="yes"/>
 </segment>
 </net>
@@
 </segment>
 </net>
+<net name="N$7" class="0">
+<segment>
+<pinref part="J1" gate="G$1" pin="1"/>
+<wire x1="99.06" y1="-17.78" x2="104.14" y2="-17.78" width="0.1524" layer="91"/>
+</segment>
+</net>

Commit message: take3
Connections:
- removed net LED: Q1.C
- net LED.C: now also Q1.C
Changed lines of the file:
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@@
 <label x="20.32" y="99.06" size="1.27" layer="95" xref="yes"/>
+</segment>
+<segment>
+<wire x1="236.22" y1="35.56" x2="236.22" y2="38.1" width="0.1524" layer="91"/>
+<label x="236.22" y="38.1" size="1.27" layer="95" rot="R180" xref="yes"/>
+<pinref part="Q1" gate="G$1" pin="C"/>
 </segment>
 </net>
@@
 </segment>
 </net>
-<net name="LED" class="0">
-<segment>
-<wire x1="236.22" y1="35.56" x2="236.22" y2="38.1" width="0.1524" layer="91"/>
-<label x="236.22" y="38.1" size="1.27" layer="95" rot="R180" xref="yes"/>
-<pinref part="Q1" gate="G$1" pin="C"/>
-</segment>
-</net>

Commit message: take3_1_24
Parts:
- J1: device LinnesLab-Connectors:CONN_07 -> LinnesLab-Connectors:CONN_07-1.27MM
- renumbered OP4 to TIA, U$4 to AD5171, U1 to AD5242
Connections:
- removed net N$7: J1.1
- net 3.3V: now also J1.4; no longer J1.3
- net A6/TIA: now also J1.6; no longer J1.5
- net D29/LED.CTRL: now also J1.5; no longer J1.6
- net GND: now also J1.3; no longer J1.2
- net SCL: now also J1.2; no longer J1.4
- net SDA: now also J1.1

Commit message: Take5
Parts:
- added C1: 100n, LinnesLab-Passives:CAPACITOR0603
- added LOGO1: REVISION.A, LinnesLab-Logos:REVISION.A
Connections:
- net GND: now also C1.1
- net VREF: now also C1.2
Other:
- note added: "AAlsaati SmartWatch PPG Circuit"
- note added: "Castellated IMU breakout"
- note added: "Connection to Digital Potentiomete for dynamic gain"
- note added: "Connection to Optical Module"
- note added: "Connection to upper board"
- note added: "Vref Generator and Bypass Capacitor"
- moved on the sheet: C10, C14, C15, C16, C19, C20, C21, J1, OP3G$1, OP3G$2, OP3G$3, R13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

Commit message: take6
Parts:
- added C2, C7, C9: 1u, LinnesLab-Passives:CAPACITOR0603
- added C3, C5: 4.7u, LinnesLab-Passives:CAPACITOR0603
- added CHRG1: MCP73831, LinnesLab-Power:MCP73831
- added LDO1: MIC5504, LinnesLab-Power:MIC5504
- added R3: 100k, LinnesLab-Passives:RESISTOR0603
- added R5: (no value), LinnesLab-Passives:RESISTOR0603
- added U3: PCF8523, LinnesLab-Clocks:PCF8523
- added XTAL2: 32.7680kHz, LinnesLab-Clocks:CRYSTALECS-.327-12.5-12-C-TR
Connections:
- new net D27/CHRG.STATUS: CHRG1.STAT, R3.1
- new net N$2: U3.OSCO, XTAL2.1
- new net N$3: U3.OSCI, XTAL2.2
- new net N$4: CHRG1.PROG, R5.2
- new net VBATT: U3.VBAT
- new net VIN1: C5.2, C7.2, CHRG1.VIN, LDO1.EN, LDO1.IN, R3.2
- new net VLIPO: C3.1, CHRG1.VBAT
- net 3.3V: now also C2.1, C9.1, LDO1.OUT, U3.VDD
- net GND: now also C2.2, C3.2, C5.1, C7.1, C9.2, CHRG1.VSS, LDO1.GND, R5.1, U3.VSS
- net SCL: now also U3.SCL
- net SDA: now also U3.SDA
Other:
- note added: "Back-up battery if desired"
- note added: "Digital Output"
- note added: "I2C Address = 0x68h"
- note added: "Power Management"
- note added: "Real-Time Clock"

Commit message: 'take8'
Parts:
- removed C3, C5: 4.7u, LinnesLab-Passives:CAPACITOR0603
- removed C7, C9: 1u, LinnesLab-Passives:CAPACITOR0603
- removed CHRG1: MCP73831, LinnesLab-Power:MCP73831
- removed LDO1: MIC5504, LinnesLab-Power:MIC5504
- removed R3: 100k, LinnesLab-Passives:RESISTOR0603
- removed R5: (no value), LinnesLab-Passives:RESISTOR0603
Connections:
- net A6/TIA renamed A5/TIA
- net A7/PPG renamed A4/PPG
- net D29/LED.CTRL renamed D30/LED.CTRL
- removed net D27/CHRG.STATUS: CHRG1.STAT, R3.1
- removed net N$4: CHRG1.PROG, R5.2
- removed net VIN1: C5.2, C7.2, CHRG1.VIN, LDO1.EN, LDO1.IN, R3.2
- removed net VLIPO: C3.1, CHRG1.VBAT
- net 3.3V: no longer C9.1, LDO1.OUT
- net GND: no longer C3.2, C5.1, C7.1, C9.2, CHRG1.VSS, LDO1.GND, R5.1
Other:
- note removed: "Digital Output"
- note removed: "Power Management"
