File: Hardware/Basic/TOP/SmartWatch-BASIC-TOP.brd (EAGLE design)
At the start: 38 x 38 mm, 52 parts, among them SW1 SWITCH.MOM, SW2 SWITCH.MOM, SW5 SWITCH.MOM, U2 NRF52832_MODULE_MDBT42, U4 PCF8523

Commit message: take 2
Parts:
- removed R8, R9: 10k, LinnesLab-Passives:R0603
- removed SW5: SWITCH.MOM, LinnesLab-Switches:TACTILE_SWITCH_SMD_6.2MM_TALL
- added C20, C6: 47p, LinnesLab-Passives:C0603
- added C5: 100n, LinnesLab-Passives:C0603
- added J3: (no value), LinnesLab-Connectors:1X06_1.27MM
- added JP2: (no value), LinnesLab-Switches:SMT-JUMPER_2_NO_SILK
- added LED5: RED, LinnesLab-LED:LED-0603
- added LED6: YELLOW, LinnesLab-LED:LED-0603
- added R1, R2: 10k, LinnesLab-Passives:R0603
- added R12, R18: 27, LinnesLab-Passives:R0603
- added R19, R20: 1k, LinnesLab-Passives:R0603
- added R21, R22: 0, LinnesLab-Passives:R0603
- added U5: FT231XS, LinnesLab-DigitalIC:SSOP20_L
- moved SW1 33.3 mm to (31.8, 3.81)
- moved SW2 27.9 mm to (20.3, 3.81)
- moved C25 10.2 mm to (10.6, 2.01)
- moved R17 10.2 mm to (12.6, 2.06)
- moved C24 6.35 mm to (8.26, 2.01)
- moved LDO2 6.35 mm to (12.6, 5.71)
- moved D4 5.68 mm to (4.70, 5.59)
- moved D5 5.08 mm to (4.67, 0.97)
- moved R16 4.58 mm to (6.96, 6.02)
- moved CHRG2 4.02 mm to (16.9, 12.8)
- moved U3 2.54 mm to (17.4, 22.6)
- moved R14 2.54 mm to (18.2, 8.61)
- moved R13 1.80 mm to (21.6, 12.9)
- moved C27 1.27 mm to (21.3, 10.2)
- moved U4 1.27 mm to (5.89, 28.2)
Connections:
- removed net BATT: R15.1, R16.2
- removed net CD1: SD2.CD1
- removed net CHRG.STAT: CHRG2.1, R14.1
- removed net CS.OLED: U3.13
- removed net DC.OLED: U3.15
- removed net RESET.OLED: U3.14
- removed net RXD: U2.21
- removed net SD.CS: SD2.2
- removed net SW1: SW1.A1, SW2.A1, SW5.A1
- removed net TXD: U2.19
- new net !CTS: JP2.2, U5.9
- new net A4/BATT: R15.1, R16.2, U2.5
- new net A6/TIA: U2.7
- new net A7/PPG: U2.8
- new net D11/SW1: SW1.A1, U2.25
- new net D15/SW2: SW2.A1, U2.29
- new net D16/CS.OLED: U2.30, U3.13
- new net D27/CHRG.STATUS: CHRG2.1, R14.1, U2.4
- new net D29/LED.CTRL: U2.6
- new net D3/RESET.OLED: U2.16, U3.14
- new net D4/DC.OLED: U2.17, U3.15
- new net D5/CD1: SD2.CD1, U2.18
- new net D7/SD.CS: SD2.2, U2.20
- new net FT3V3: U5.13
- new net N$23: R12.2, U5.12
- new net N$24: R18.2, U5.11
- new net N$25: LED5.C, R19.2
- new net N$26: LED6.C, R20.2
- new net RXD.FT: R22.1, U5.4
- new net RXD.NRF: R21.2, U2.21
- new net RXLED: R19.1, U5.17
- new net TXD.FT: R21.1, U5.20
- new net TXD.NRF: R22.2, U2.19
- new net TXLED: R20.1, U5.10
- net 3.3V: now also C5.2, LED5.A, LED6.A, R1.2, R2.2, U5.14, U5.3; no longer R8.2, R9.2
- net DTR: now also U5.1
- net GND: now also C20.1, C5.1, C6.2, JP2.1, U5.16, U5.6; no longer SW5.B1, SW5.B2
- net SCL: now also R2.1; no longer R8.1
- net SDA: now also R1.1; no longer R9.1
- net USB+: now also C6.1, R18.1
- net USB-: now also C20.2, R12.1
- net V_USB: now also U5.15

Commit message: Take5
Parts:
- removed C24, C25: 1u, LinnesLab-Passives:C0603
- removed C26, C27: 4.7u, LinnesLab-Passives:C0603
- removed C6: 47p, LinnesLab-Passives:C0603
- removed C8: (no value), LinnesLab-Passives:C0603
- removed CHRG2: MCP73831, LinnesLab-Power:SOT23-5
- removed CORTEX1: CORTEX_DEBUG_PTH, LinnesLab-Connectors:2X5-PTH-1.27MM
- removed D4, D5: (no value), LinnesLab-DiscreteSemi:USC
- removed J3: (no value), LinnesLab-Connectors:1X06_1.27MM
- removed JP2: (no value), LinnesLab-Switches:SMT-JUMPER_2_NO_SILK
- removed L2: 10u, LinnesLab-Passives:L0603
- removed LDO2: MIC5504, LinnesLab-Power:SOT23-5
- removed LED5: RED, LinnesLab-LED:LED-0603
- removed LED6: YELLOW, LinnesLab-LED:LED-0603
- removed R19, R20: 1k, LinnesLab-Passives:R0603
- removed R21, R22: 0, LinnesLab-Passives:R0603
- removed R6: 10k, LinnesLab-Passives:R0603
- removed U5: FT231XS, LinnesLab-DigitalIC:SSOP20_L
- removed XTAL3: 32.7680kHz, LinnesLab-Clocks:2-SMD.NOLEAD.2.0MMTO1.2MM
- added C1, C21: 1u, LinnesLab-Passives:C0603
- added C3, C4: (no value), LinnesLab-Passives:C0603
- added CHRG1: MCP73831, LinnesLab-Power:SOT23-5
- added D2, D3: (no value), LinnesLab-DiscreteSemi:USC
- added DEBUG1: CORTEX_DEBUG_PTH, LinnesLab-Connectors:2X5-PTH-1.27MM
- added J1: (no value), LinnesLab-Connectors:1X02
- added JP1: (no value), LinnesLab-Switches:SMT-JUMPER_2_NO_SILK
- added L1: 10u, LinnesLab-Passives:L0603
- added LDO1: MIC5504, LinnesLab-Power:SOT23-5
- added LED1: RED, LinnesLab-LED:LED-0603
- added LED2: BLUE, LinnesLab-LED:LED-0603
- added R10: 10k, LinnesLab-Passives:R0603
- added R11: 27, LinnesLab-Passives:R0603
- added R8, R9: 100k, LinnesLab-Passives:R0603
- added U1: NRF52832_MODULE_MDBT42, LinnesLab-Microcontrollers:BLE_MODULE_RAYTAC_MDBT42
- added XTAL1: 32.768kHz, LinnesLab-Clocks:2-SMD.NOLEAD.2.0MMTO1.2MM
- C10: value 300p -> 4.7u
- C11: value 300p -> 47p
- C12: value 10u -> 100n; device LinnesLab-Passives:C0805 -> LinnesLab-Passives:C0603
- C13: value 2.2uF -> 47p; device LinnesLab-Passives:C0402 -> LinnesLab-Passives:C0603
- C15: value 2.2uF -> 10uF; device LinnesLab-Passives:C0402 -> LinnesLab-Passives:C0603
- C16: value 10uF -> 2.2uF; device LinnesLab-Passives:C0603 -> LinnesLab-Passives:C0402
- C2: value 1u -> 10u; device LinnesLab-Passives:C0603 -> LinnesLab-Passives:C0805
- C20: value 47p -> 2.2uF; device LinnesLab-Passives:C0603 -> LinnesLab-Passives:C0402
- C5: value 100n -> 4.7u
- C9: value (none) -> 1u
- J2: device LinnesLab-Connectors:1X02 -> LinnesLab-Connectors:1X07_1.27MM
- LED4: value BLUE -> YELLOW
- R13: value (none) -> 10k
- R14, R15: value 100k -> 1k
- R16: value 100k -> 390k
- R17: value 100k -> 0
- R18: value 27 -> 0
- R3: value 1k -> 100k
- R5: value 10k -> (none)
- R7: value 390k -> 1k
- SW1, SW2: value SWITCH.MOM -> (none); device LinnesLab-Switches:TACTILE_SWITCH_SMD_6.2MM_TALL -> LinnesLab-Switches:BUTTON-GULLWING
- SW3, SW4: value (none) -> SWITCH.MOM; device LinnesLab-Switches:BUTTON-GULLWING -> LinnesLab-Switches:TACTILE_SWITCH_SMD_6.2MM_TALL
- U2: value NRF52832_MODULE_MDBT42 -> FT231XS; device LinnesLab-Microcontrollers:BLE_MODULE_RAYTAC_MDBT42 -> LinnesLab-DigitalIC:SSOP20_L
- U3: value (none) -> PCF8523; device LinnesLab-Displays:UG-2864HSWEG01_0.96IN_NO-WRAPAROUND -> LinnesLab-Clocks:SO8
- U4: value PCF8523 -> (none); device LinnesLab-Clocks:SO8 -> LinnesLab-Displays:UG-2864HSWEG01_0.96IN_NO-WRAPAROUND
- XTAL2: value 32.768kHz -> 32.7680kHz
- moved R12 92.8 mm to (2.05, -37.4), turned to 180 degrees
- moved R18 89.4 mm to (-4.37, -28.0)
- moved C14 76.3 mm to (-7.84, -30.7)
- moved C5 73.2 mm to (10.6, 5.49), flipped to the bottom
- moved U2 71.1 mm to (-3.23, -33.7), turned to 270 degrees
- moved LED4 68.4 mm to (5.92, -30.1), turned to 180 degrees
- moved LED3 68.4 mm to (6.17, -32.7), turned to 180 degrees
- moved C20 64.6 mm to (13.9, 22.0), turned to 270 degrees
- moved C11 61.5 mm to (3.29, -34.4)
- moved C13 61.4 mm to (5.59, -37.4), turned to 0 degrees
- moved R2 53.5 mm to (6.40, 36.0)
- moved R1 50.3 mm to (10.0, 35.7), turned to 180 degrees
- moved U3 46.9 mm to (51.3, 55.0)
- moved R14 44.3 mm to (2.39, -32.7)
- moved XTAL2 42.8 mm to (46.3, 56.1), turned to 90 degrees
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- renumbered SD2 to SD1, USB2 to USB1
Connections:
- net !CTS: now also JP1.2, U2.9; no longer JP2.2, U5.9
- net 3.3V: now also C14.2, C2.2, C20.2, C21.1, C9.1, D3.-, DEBUG1.1, J2.4, LDO1.5, LED3.A, LED4.A, R10.2, U1.11, U2.14, U2.3, U3.8, U4.6, U4.9; no longer C12.2, C17.2, C2.1, C25.1, C5.2, CORTEX1.1, D1.-, LDO2.5, LED5.A, LED6.A, R17.2, R5.2, U2.11, U3.6, U3.9, U4.8, U5.14, U5.3
- net A4/BATT: now also R8.1, R9.2, U1.5; no longer R15.1, R16.2, U2.5
- net A6/TIA: now also J2.6, U1.7; no longer U2.7
- net A7/PPG: now also J2.7, U1.8; no longer U2.8
- net D11/SW1: now also SW3.A1, U1.25; no longer SW1.A1, U2.25
- net D15/SW2: now also SW4.A1, U1.29; no longer SW2.A1, U2.29
- net D16/CS.OLED: now also U1.30, U4.13; no longer U2.30, U3.13
- net D27/CHRG.STATUS: now also CHRG1.1, R3.1, U1.4; no longer CHRG2.1, R14.1, U2.4
- net D29/LED.CTRL: now also J2.5, U1.6; no longer U2.6
- net D3/RESET.OLED: now also U1.16, U4.14; no longer U2.16, U3.14
- net D4/DC.OLED: now also U1.17, U4.15; no longer U2.17, U3.15
- net D5/CD1: now also U1.18; no longer U2.18
- net D7/SD.CS: now also U1.20; no longer U2.20
- net DFU: now also SW1.3, U1.34; no longer SW3.3, U2.34
- net DTR: now also C12.1, U2.1; no longer C14.1, U5.1
- net FRST: now also U1.38; no longer U2.38
- net FT3V3: now also U2.13; no longer U5.13
- net GND: now also C1.2, C11.1, C13.2, C14.1, C15.1, C2.1, C21.2, C3.1, C4.2, C7.1, CHRG1.2, DEBUG1.3, DEBUG1.5, DEBUG1.7, DEBUG1.9, J1.1, J2.3, JP1.1, LDO1.2, LED1.C, LED2.C, R16.2, R5.1, R9.1, SW1.1, SW2.3, SW3.B1, SW4.B1, U1.1, U1.12, U1.24, U1.39, U2.16, U2.6, U3.4, U4.1, U4.10, U4.12, U4.29, U4.30, U4.8; no longer C11.2, C12.1, C16.1, C18.1, C2.2, C24.1, C25.2, C26.2, C27.1, C6.2, C7.2, C8.1, CHRG2.2, CORTEX1.3, CORTEX1.5, CORTEX1.7, CORTEX1.9, J2.1, JP2.1, LDO2.2, LED3.C, LED4.C, R16.1, R17.1, R6.1, R7.2, SW1.B1, SW1.B2, SW2.B1, SW2.B2, SW3.1, SW4.3, U2.1, U2.12, U2.24, U2.39, U3.1, U3.10, U3.12, U3.29, U3.30, U3.8, U4.4, U5.16, U5.6
- net LED1: now also R4.2, U1.31; no longer R3.2, U2.31
- net LED2: now also R7.2, U1.33; no longer R4.2, U2.33
- net MISO: now also U1.28; no longer U2.28
- net MOSI: now also U1.27, U4.19; no longer U2.27, U3.19
- net N$1: now also R13.2, U4.11; no longer R6.2, U3.11
- net N$10: now also LED2.A, R7.1; no longer LED4.A, R4.1
- net N$11: now also L1.1, U1.10; no longer L2.1, U2.10
- net N$12: now also C1.1, L1.2, U1.9; no longer C7.1, L2.2, U2.9
- net N$13: now also C15.2, U4.28; no longer C16.2, U3.28
- net N$14: now also DEBUG1.8; no longer CORTEX1.8
- net N$15: now also C17.2, U4.27; no longer C18.2, U3.27
- net N$17: now also CHRG1.5, R5.2; no longer CHRG2.5, R13.2
- net N$19: now also U3.2, XTAL2.P$1; no longer U4.2, XTAL3.P$1
- net N$2: now also R16.1, U4.26; no longer R7.1, U3.26
- net N$20: now also U3.1, XTAL2.P$2; no longer U4.1, XTAL3.P$2
- net N$23: now also R11.2, U2.12; no longer R12.2, U5.12
- net N$24: now also R12.2, U2.11; no longer R18.2, U5.11
- net N$25: now also LED3.C, R14.2; no longer LED5.C, R19.2
- net N$26: now also LED4.C, R15.2; no longer LED6.C, R20.2
- net N$3: now also C18.2, U4.2; no longer C13.2, U3.2
- net N$4: now also C3.2, U1.13, XTAL1.P$1; no longer C8.2, U2.13, XTAL2.P$1
- net N$5: now also C18.1, U4.3; no longer C13.1, U3.3
- net N$6: now also C4.1, U1.14, XTAL1.P$2; no longer C9.1, U2.14, XTAL2.P$2
- net N$7: now also C16.2, U4.4; no longer C15.2, U3.4
- net N$8: now also C16.1, U4.5; no longer C15.1, U3.5
- net N$9: now also LED1.A, R4.1; no longer LED3.A, R3.1
- net P0.09/NFC1: now also U1.22; no longer C11.1, U2.22
- net P0.10/NFC2: now also U1.23; no longer C10.1, U2.23
- net RESET: now also C12.2, D3.+, DEBUG1.10, R10.1, SW2.1, U1.35; no longer C14.2, CORTEX1.10, D1.+, R5.1, SW4.1, U2.35
- net RXD.FT: now also R18.1, U2.4; no longer R22.1, U5.4
- net RXD.NRF: now also R17.2, U1.21; no longer R21.2, U2.21
- net RXLED: now also R14.1, U2.17; no longer R19.1, U5.17
- net SCK: now also U1.26, U4.18; no longer U2.26, U3.18
- net SCL: now also J2.2, U1.3, U3.6; no longer U2.3, U4.6
- net SDA: now also J2.1, U1.2, U3.5; no longer U2.2, U4.5
- net SWCLK: now also DEBUG1.4, U1.36; no longer CORTEX1.4, U2.36
- net SWDIO: now also DEBUG1.2, U1.37; no longer CORTEX1.2, U2.37
- net SWO: now also DEBUG1.6, U1.32; no longer CORTEX1.6, U2.32
- net TXD.FT: now also R17.1, U2.20; no longer R21.1, U5.20
- net TXD.NRF: now also R18.2, U1.19; no longer R22.2, U2.19
- net TXLED: now also R15.1, U2.10; no longer R20.1, U5.10
- net USB+: now also C13.1, R12.1; no longer C6.1, R18.1
- net USB-: now also C11.2, R11.1; no longer C20.2, R12.1
- net VBATT: now also U3.3; no longer U4.3
- net VIN: now also C5.2, C7.2, CHRG1.4, D1.-, D2.-, LDO1.1, LDO1.3, R3.2; no longer C24.2, C27.2, CHRG2.4, D4.-, D5.-, LDO2.1, LDO2.3, R14.2
- net VLIPO: now also C10.1, CHRG1.3, D1.+, J1.2, R8.2; no longer C26.1, CHRG2.3, D4.+, J2.2, R15.2
- net V_USB: now also D2.+, U2.15; no longer D5.+, U5.15
Routing:
- net GND: track 0.00 -> 26.8 mm, vias 0 -> 14
- net VLIPO: track 0.00 -> 21.8 mm
- net VIN: track 0.00 -> 14.9 mm
- net N$6: track 0.00 -> 6.89 mm
- net N$4: track 0.00 -> 6.00 mm
- net N$17: track 0.00 -> 5.30 mm
- net N$5: track 0.00 -> 4.74 mm
- net N$12: track 0.00 -> 4.53 mm
- net N$8: track 0.00 -> 4.28 mm
- net 3.3V: track 0.00 -> 4.28 mm, vias 0 -> 1
- net N$15: track 0.00 -> 3.65 mm
- net N$3: track 0.00 -> 3.15 mm
- net N$1: track 0.00 -> 2.74 mm
- net N$7: track 0.00 -> 2.69 mm
- net N$19: track 0.00 -> 2.43 mm
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- added copper zone on layer 1, net 3.3V
- added copper zone on layer 16, net GND

Commit message: take7
Parts:
- removed C10, C5: 4.7u, LinnesLab-Passives:C0603
- removed C21, C7, C9: 1u, LinnesLab-Passives:C0603
- removed CHRG1: MCP73831, LinnesLab-Power:SOT23-5
- removed LDO1: MIC5504, LinnesLab-Power:SOT23-5
- removed R3: 100k, LinnesLab-Passives:R0603
- removed R5: (no value), LinnesLab-Passives:R0603
- removed SD1: (no value), LinnesLab-Connectors:MICROSD
- removed U3: PCF8523, LinnesLab-Clocks:SO8
- removed XTAL2: 32.7680kHz, LinnesLab-Clocks:2-SMD.NOLEAD.2.0MMTO1.2MM
- C17: device LinnesLab-Passives:C0402 -> LinnesLab-Passives:C0603
- moved JP1 45.5 mm to (1.79, 1.80), turned to 90 degrees
- moved R18 45.2 mm to (19.4, 10.4)
- moved R17 41.4 mm to (19.3, 8.59)
- moved R12 41.3 mm to (11.4, 2.81)
- moved R11 41.2 mm to (11.6, 4.22)
- moved R14 41.2 mm to (11.8, 7.40)
- moved C13 41.1 mm to (14.8, 2.62)
- moved C11 40.8 mm to (11.6, 5.55)
- moved LED3 40.7 mm to (15.3, 7.01)
- moved U2 40.6 mm to (6.31, 5.75)
- moved C14 40.3 mm to (1.49, 8.51)
- moved LED4 40.2 mm to (15.1, 9.06)
- moved R15 39.9 mm to (11.8, 8.78)
- moved SW2 35.8 mm to (34.9, 14.4), turned to 270 degrees
- moved R10 35.5 mm to (34.9, 11.3), turned to 180 degrees
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Connections:
- removed net A4/BATT: R8.1, R9.2, U1.5
- removed net A6/TIA: J2.6, U1.7
- removed net A7/PPG: J2.7, U1.8
- removed net CD2: SD1.CD2
- removed net D29/LED.CTRL: J2.5, U1.6
- removed net N$17: CHRG1.5, R5.2
- removed net N$19: U3.2, XTAL2.P$1
- removed net N$20: U3.1, XTAL2.P$2
- removed net VBATT: U3.3
- new net A4/PPG: J2.7, U1.5
- new net A5/TIA: J2.6, U1.6
- new net A7/BATT: R8.1, R9.2, U1.8
- new net D30/LED.CTRL: J2.5, U1.7
- net 3.3V: no longer C21.1, C9.1, LDO1.5, SD1.4, U3.8
- net D27/CHRG.STATUS: no longer CHRG1.1, R3.1
- net D5/CD1: no longer SD1.CD1
- net D7/SD.CS: no longer SD1.2
- net GND: no longer C10.2, C21.2, C5.1, C7.1, C9.2, CHRG1.2, LDO1.2, R5.1, SD1.6, SD1.MT1, SD1.MT2, U3.4
- net MISO: no longer SD1.7
- net MOSI: no longer SD1.3
- net SCK: no longer SD1.5
- net SCL: no longer U3.6
- net SDA: no longer U3.5
- net VIN: no longer C5.2, C7.2, CHRG1.4, LDO1.1, LDO1.3, R3.2
- net VLIPO: no longer C10.1, CHRG1.3
Routing:
- net 3.3V: track 4.28 -> 42.5 mm, vias 1 -> 0
- net RESET: track 0.00 -> 30.6 mm, vias 0 -> 1
- net RXD.NRF: track 0.00 -> 28.5 mm, vias 0 -> 2
- net D15/SW2: track 0.00 -> 24.4 mm, vias 0 -> 2
- net TXD.NRF: track 0.00 -> 23.6 mm, vias 0 -> 2
- net A7/BATT: track 0.00 -> 23.1 mm, vias 0 -> 2
- net SDA: track 0.00 -> 22.4 mm, vias 0 -> 1
- net GND: track 26.8 -> 48.4 mm, vias 14 -> 23
- net SCL: track 0.00 -> 20.5 mm, vias 0 -> 1
- net D11/SW1: track 0.00 -> 20.3 mm
- net D16/CS.OLED: track 0.00 -> 18.8 mm, vias 0 -> 2
- net USB-: track 2.04 -> 20.6 mm, vias 0 -> 1
- net RXD.FT: track 0.57 -> 17.4 mm
- net SCK: track 0.00 -> 16.2 mm, vias 0 -> 2
- net MOSI: track 0.00 -> 15.1 mm, vias 0 -> 2
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
Commit message: take 8
Parts:
- added C5, C6: 4.7u, LinnesLab-Passives:C0603
- added C7, C9: 1u, LinnesLab-Passives:C0603
- added CHRG1: MCP73831, LinnesLab-Power:SOT23-5
- added LDO1: MIC5504, LinnesLab-Power:SOT23-5
- added R3: 100k, LinnesLab-Passives:R0603
- added R5: (no value), LinnesLab-Passives:R0603
- moved D3 1.94 mm to (35.2, 7.89)
- moved C12 1.66 mm to (35.1, 9.61)
- moved R2 1.46 mm to (3.14, 32.8)
- moved R1 1.42 mm to (1.59, 32.8)
- moved JP1 1.34 mm to (1.64, 3.13)
- moved J1 0.29 mm to (2.10, 15.6)
- moved C14 0.20 mm to (1.64, 8.39)
- moved C20 0.13 mm to (13.5, 22.2)
- moved R9 0.12 mm to (1.82, 18.9)
- moved C4 0.12 mm to (18.0, 23.5)
- moved R8 0.11 mm to (3.42, 18.8)
- moved USB1 0.10 mm to (3.34, 5.89)
Connections:
- new net N$16: CHRG1.5, R5.2
- net 3.3V: now also C9.1, LDO1.5
- net D27/CHRG.STATUS: now also CHRG1.1, R3.1
- net GND: now also C5.2, C6.1, C7.1, C9.2, CHRG1.2, LDO1.2, R5.1
- net VIN: now also C6.2, C7.2, CHRG1.4, LDO1.1, LDO1.3, R3.2
- net VLIPO: now also C5.1, CHRG1.3
Routing:
- net VIN: track 5.69 -> 45.4 mm, vias 0 -> 1
- net DTR: track 0.00 -> 38.7 mm
- net D27/CHRG.STATUS: track 0.00 -> 33.5 mm, vias 0 -> 3
- net GND: track 48.4 -> 74.3 mm, vias 23 -> 28
- net VLIPO: track 20.5 -> 31.5 mm, vias 0 -> 1
- net A7/BATT: track 23.1 -> 27.9 mm
- net N$16: track 0.00 -> 1.76 mm
- net SCL: track 20.5 -> 21.6 mm
- net SDA: track 22.4 -> 23.5 mm
- net 3.3V: track 42.5 -> 41.5 mm
- net RESET: track 30.6 -> 31.4 mm
- net N$11: track 5.59 -> 6.14 mm
- net N$12: track 5.77 -> 6.31 mm

Commit message: take8
Parts:
- moved C11 0.58 mm to (12.2, 5.67)
- moved R14 0.11 mm to (11.8, 7.30)
Routing:
- net VLIPO: track 31.5 -> 32.2 mm
- net USB-: track 20.6 -> 21.2 mm

Commit message: 'take8'
Parts:
- removed C19, C20: 2.2uF, LinnesLab-Passives:C0402
- removed R18: 0, LinnesLab-Passives:R0603
- removed U4: (no value), LinnesLab-Displays:UG-2864HSWEG01_0.96IN_NO-WRAPAROUND
- added C10: 2.2uF, LinnesLab-Passives:C0402
- added C8: 4.7u, LinnesLab-Passives:C0603
- added R6: 1k, LinnesLab-Passives:R0603
- added U3: FT231XS, LinnesLab-DigitalIC:SSOP20_L
- C11: value 47p -> 2.2uF
- C12, C14: value 100n -> 2.2uF; device LinnesLab-Passives:C0603 -> LinnesLab-Passives:C0402
- C13: value 47p -> 2.2uF; device LinnesLab-Passives:C0603 -> LinnesLab-Passives:C0402
- C15: value 10uF -> 47p
- C16: value 2.2uF -> 47p; device LinnesLab-Passives:C0402 -> LinnesLab-Passives:C0603
- C17: value 2.2uF -> 100n
- C18: value 2.2uF -> 100n; device LinnesLab-Passives:C0402 -> LinnesLab-Passives:C0603
- C6: value 4.7u -> 1u
- C9: value 1u -> 10uF
- R10: value 10k -> 390k
- R13: value 10k -> 1k
- R15: value 1k -> 0
- R16: value 390k -> 0
- R17: value 0 -> 10k
- R7: value 1k -> 100k
- R9: value 100k -> 10k
- SW2: value (none) -> SWITCH.MOM; device LinnesLab-Switches:BUTTON-GULLWING -> LinnesLab-Switches:TACTILE_SWITCH_SMD_6.2MM_TALL
- SW4: value SWITCH.MOM -> (none); device LinnesLab-Switches:TACTILE_SWITCH_SMD_6.2MM_TALL -> LinnesLab-Switches:BUTTON-GULLWING
- U2: value FT231XS -> (none); device LinnesLab-DigitalIC:SSOP20_L -> LinnesLab-Displays:UG-2864HSWEG01_0.96IN_NO-WRAPAROUND
- moved R7 32.0 mm to (3.42, 18.8), turned to 270 degrees
- moved C12 30.1 mm to (7.87, 22.5), turned to 270 degrees
- moved C18 30.1 mm to (35.1, 9.61), turned to 0 degrees
- moved C17 28.9 mm to (1.64, 8.39), turned to 270 degrees
- moved C9 22.5 mm to (29.6, 18.8), turned to 90 degrees
- moved C15 21.8 mm to (12.2, 5.67), turned to 0 degrees
- moved C16 20.3 mm to (14.8, 2.62), turned to 0 degrees
- moved C13 19.6 mm to (12.1, 22.1), turned to 270 degrees
- moved U2 18.9 mm to (18.4, 20.3), turned to 0 degrees
- moved C14 18.2 mm to (13.5, 22.2)
- moved SW2 16.8 mm to (21.8, 3.96), turned to 180 degrees
- moved R17 15.8 mm to (34.9, 11.3), turned to 180 degrees
- moved R13 15.4 mm to (11.8, 7.30), turned to 0 degrees
- moved C11 15.1 mm to (26.7, 9.94), turned to 180 degrees
- moved R16 14.6 mm to (19.4, 10.4), turned to 0 degrees
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Connections:
- net !CTS: now also U3.9; no longer U2.9
- net 3.3V: now also C13.2, C17.2, C7.1, R17.2, U2.6, U2.9, U3.14, U3.3; no longer C19.2, C20.2, C9.1, R10.2, U2.14, U2.3, U4.6, U4.9
- net A7/BATT: now also R7.1, R8.2; no longer R8.1, R9.2
- net D11/SW1: now also SW2.A1; no longer SW3.A1
- net D15/SW2: now also SW3.A1; no longer SW4.A1
- net D16/CS.OLED: now also U2.13; no longer U4.13
- net D3/RESET.OLED: now also U2.14; no longer U4.14
- net D4/DC.OLED: now also U2.15; no longer U4.15
- net DTR: now also C18.1, U3.1; no longer C12.1, U2.1
- net FT3V3: now also U3.13; no longer U2.13
- net GND: now also C13.1, C16.2, C5.1, C7.2, C8.2, C9.1, R10.2, R8.1, SW2.B1, SW4.3, U2.1, U2.10, U2.12, U2.29, U2.30, U2.8, U3.16, U3.6; no longer C13.2, C19.1, C20.1, C5.2, C7.1, C9.2, R13.1, R16.2, SW2.3, SW4.B1, U2.16, U2.6, U4.1, U4.10, U4.12, U4.29, U4.30, U4.8
- net LED2: now also R6.2; no longer R7.2
- net MOSI: now also U2.19; no longer U4.19
- net N$1: now also R9.2, U2.11; no longer R13.2, U4.11
- net N$10: now also R6.1; no longer R7.1
- net N$13: now also C9.2, U2.28; no longer C15.2, U4.28
- net N$15: now also C11.2, U2.27; no longer C17.2, U4.27
- net N$2: now also R10.1, U2.26; no longer R16.1, U4.26
- net N$23: now also U3.12; no longer U2.12
- net N$24: now also U3.11; no longer U2.11
- net N$25: now also R13.2; no longer R14.2
- net N$26: now also R14.2; no longer R15.2
- net N$3: now also C12.2, U2.2; no longer C18.2, U4.2
- net N$5: now also C12.1, U2.3; no longer C18.1, U4.3
- net N$7: now also C10.2, U2.4; no longer C16.2, U4.4
- net N$8: now also C10.1, U2.5; no longer C16.1, U4.5
- net RESET: now also C18.2, R17.1, SW4.1; no longer C12.2, R10.1, SW2.1
- net RXD.FT: now also R16.1, U3.4; no longer R18.1, U2.4
- net RXD.NRF: now also R15.2; no longer R17.2
- net RXLED: now also R13.1, U3.17; no longer R14.1, U2.17
- net SCK: now also U2.18; no longer U4.18
- net TXD.FT: now also R15.1, U3.20; no longer R17.1, U2.20
- net TXD.NRF: now also R16.2; no longer R18.2
- net TXLED: now also R14.1, U3.10; no longer R15.1, U2.10
- net USB+: now also C16.1; no longer C13.1
- net USB-: now also C15.2; no longer C11.2
- net VIN: now also C5.2; no longer C7.2
- net VLIPO: now also C8.1, R7.2; no longer C5.1, R8.2
- net V_USB: now also U3.15; no longer U2.15
Routing:
- net GND: track 74.7 -> 80.0 mm
- net D15/SW2: track 24.4 -> 27.5 mm
- net N$15: track 6.55 -> 9.43 mm
- net DTR: track 38.7 -> 40.0 mm, vias 0 -> 2
Other:
- board text added: "+"
- board text added: "-"
