File: Hardware/Basic/TOP/SmartWatch-BASIC-TOP.sch (EAGLE design)
At the start: 52 parts, among them SW1 SWITCH.MOM, SW2 SWITCH.MOM, SW5 SWITCH.MOM, U2 NRF52832_MODULE_MDBT42, U4 PCF8523

Commit message: take 2
Parts:
- removed R8, R9: 10k, LinnesLab-Passives:RESISTOR0603
- removed SW5: SWITCH.MOM, LinnesLab-Switches:SWITCH.MOM
- added C20, C6: 47p, LinnesLab-Passives:CAPACITOR0603
- added C5: 100n, LinnesLab-Passives:CAPACITOR0603
- added J3: (no value), LinnesLab-Connectors:CONN_061.27MM
- added JP2: (no value), LinnesLab-Switches:JUMPER-SMT_2_NO_SILK
- added LED5: RED, LinnesLab-LED:LED0603
- added LED6: YELLOW, LinnesLab-LED:LED0603
- added R1, R2: 10k, LinnesLab-Passives:RESISTOR0603
- added R12, R18: 27, LinnesLab-Passives:RESISTOR0603
- added R19, R20: 1k, LinnesLab-Passives:RESISTOR0603
- added R21, R22: 0, LinnesLab-Passives:RESISTOR0603
- added U5: FT231XS, LinnesLab-DigitalIC:FT231XS
Connections:
- removed net BATT: R15.1, R16.2
- removed net CD1: SD2.CARD_DETECT
- removed net CHRG.STAT: CHRG2.STAT, R14.1
- removed net CS.OLED: U3./CS
- removed net DC.OLED: U3.DC/I2C_SA0
- removed net RESET.OLED: U3./RES
- removed net RXD: U2.P0.08
- removed net SD.CS: SD2.CS
- removed net SW1: SW1.1, SW2.1, SW5.1
- removed net TXD: U2.P0.06
- new net !CTS: JP2.2, U5.!CTS
- new net A4/BATT: R15.1, R16.2, U2.P0.28/AIN4
- new net A6/TIA: U2.P0.30/AIN6
- new net A7/PPG: U2.P0.31/AIN7
- new net D11/SW1: SW1.1, U2.P0.11
- new net D15/SW2: SW2.1, U2.P0.15
- new net D16/CS.OLED: U2.P0.16, U3./CS
- new net D27/CHRG.STATUS: CHRG2.STAT, R14.1, U2.P0.27
- new net D29/LED.CTRL: U2.P0.29/AIN5
- new net D3/RESET.OLED: U2.P0.03/AIN1, U3./RES
- new net D4/DC.OLED: U2.P0.04/AIN2, U3.DC/I2C_SA0
- new net D5/CD1: SD2.CARD_DETECT, U2.P0.05/AIN3
- new net D7/SD.CS: SD2.CS, U2.P0.07
- new net FT3V3: U5.3V3OUT
- new net N$23: R12.2, U5.USBDM
- new net N$24: R18.2, U5.USBDP
- new net N$25: LED5.C, R19.2
- new net N$26: LED6.C, R20.2
- new net RXD.FT: R22.1, U5.RXD
- new net RXD.NRF: R21.2, U2.P0.08
- new net RXLED: R19.1, U5.CBUS1
- new net TXD.FT: R21.1, U5.TXD
- new net TXD.NRF: R22.2, U2.P0.06
- new net TXLED: R20.1, U5.CBUS2
- net 3.3V: now also C5.2, LED5.A, LED6.A, R1.2, R2.2, U5.!RESET, U5.VCCIO; no longer R8.2, R9.2
- net DTR: now also U5.!DTR
- net GND: now also C20.1, C5.1, C6.2, JP2.1, U5.GND@16, U5.GND@6; no longer SW5.3, SW5.4
- net SCL: now also R2.1; no longer R8.1
- net SDA: now also R1.1; no longer R9.1
- net USB+: now also C6.1, R18.1
- net USB-: now also C20.2, R12.1
- net V_USB: now also U5.VCC
Other:
- note added: "Digital Output"
- note added: "FTDI serial-to-USB Converter"
- note added: "I don't remember if CTS needs to be grounded or left floating so here's a jumper to ground so it can be configued either way dynamically."
- note added: "TXD goes to RX on the other device RXD goes to TX on the other device"

Commit message: Take5
Parts:
- removed C24, C25: 1u, LinnesLab-Passives:CAPACITOR0603
- removed C26, C27: 4.7u, LinnesLab-Passives:CAPACITOR0603
- removed C6: 47p, LinnesLab-Passives:CAPACITOR0603
- removed D4: (no value), LinnesLab-DiscreteSemi:SCHOTTKY-USC
- removed J3: (no value), LinnesLab-Connectors:CONN_061.27MM
- removed LED5: RED, LinnesLab-LED:LED0603
- removed LED6: YELLOW, LinnesLab-LED:LED0603
- removed R19, R20: 1k, LinnesLab-Passives:RESISTOR0603
- removed R21, R22: 0, LinnesLab-Passives:RESISTOR0603
- removed R6: 10k, LinnesLab-Passives:RESISTOR0603
- removed U5: FT231XS, LinnesLab-DigitalIC:FT231XS
- removed XTAL3: 32.7680kHz, LinnesLab-Clocks:CRYSTALECS-.327-12.5-12-C-TR
- added C1, C21: 1u, LinnesLab-Passives:CAPACITOR0603
- added C4: (no value), LinnesLab-Passives:CAPACITOR0603
- added D3: (no value), LinnesLab-DiscreteSemi:SCHOTTKY-USC
- added J1: (no value), LinnesLab-Connectors:CONN_02
- added LED1: RED, LinnesLab-LED:LED0603
- added LED2: BLUE, LinnesLab-LED:LED0603
- added R10: 10k, LinnesLab-Passives:RESISTOR0603
- added R11: 27, LinnesLab-Passives:RESISTOR0603
- added R8, R9: 100k, LinnesLab-Passives:RESISTOR0603
- added U1: NRF52832_MODULE_MDBT42, LinnesLab-Microcontrollers:NRF52832_MODULE_MDBT42
- added XTAL1: 32.768kHz, LinnesLab-Clocks:CRYSTALECS-.327-12.5-12-C-TR
- C10: value 300p -> 4.7u
- C11: value 300p -> 47p
- C12: value 10u -> 100n; device LinnesLab-Passives:CAPACITOR0805 -> LinnesLab-Passives:CAPACITOR0603
- C13: value 2.2uF -> 47p; device LinnesLab-Passives:CAPACITOR0402 -> LinnesLab-Passives:CAPACITOR0603
- C15: value 2.2uF -> 10uF; device LinnesLab-Passives:CAPACITOR0402 -> LinnesLab-Passives:CAPACITOR0603
- C16: value 10uF -> 2.2uF; device LinnesLab-Passives:CAPACITOR0603 -> LinnesLab-Passives:CAPACITOR0402
- C2: value 1u -> 10u; device LinnesLab-Passives:CAPACITOR0603 -> LinnesLab-Passives:CAPACITOR0805
- C20: value 47p -> 2.2uF; device LinnesLab-Passives:CAPACITOR0603 -> LinnesLab-Passives:CAPACITOR0402
- C5: value 100n -> 4.7u
- C9: value (none) -> 1u
- J2: device LinnesLab-Connectors:CONN_02 -> LinnesLab-Connectors:CONN_07-1.27MM
- LED4: value BLUE -> YELLOW
- R13: value (none) -> 10k
- R14, R15: value 100k -> 1k
- R16: value 100k -> 390k
- R17: value 100k -> 0
- R18: value 27 -> 0
- R3: value 1k -> 100k
- R5: value 10k -> (none)
- R7: value 390k -> 1k
- SW1, SW2: value SWITCH.MOM -> (none); device LinnesLab-Switches:SWITCH.MOM -> LinnesLab-Switches:SPST-PTS830GG140-COPY.1-3
- SW3, SW4: value (none) -> SWITCH.MOM; device LinnesLab-Switches:SPST-PTS830GG140-COPY.1-3 -> LinnesLab-Switches:SWITCH.MOM
- U2: value NRF52832_MODULE_MDBT42 -> FT231XS; device LinnesLab-Microcontrollers:NRF52832_MODULE_MDBT42 -> LinnesLab-DigitalIC:FT231XS
- U3: value (none) -> PCF8523; device LinnesLab-Displays:DISP_OLED_UG-2864HSWEG01-NO-WRAPAROUND -> LinnesLab-Clocks:PCF8523; DIGIKEY (none) -> 568-5306-1-ND; I2C_ADDRESS (none) -> 0x68h; MFN (none) -> PCF8523T/1,118; MFN_MANUFACTURER (none) -> NXP USA Inc.
- U4: value PCF8523 -> (none); device LinnesLab-Clocks:PCF8523 -> LinnesLab-Displays:DISP_OLED_UG-2864HSWEG01-NO-WRAPAROUND; DIGIKEY 568-5306-1-ND -> (none); I2C_ADDRESS 0x68h -> (none); MFN PCF8523T/1,118 -> (none); MFN_MANUFACTURER NXP USA Inc. -> (none)
- XTAL2: value 32.768kHz -> 32.7680kHz; FREQ (none) -> 32.7680KHZ
- renumbered C8 to C3, CHRG2 to CHRG1, CORTEX1 to DEBUG1, D5 to D2, JP2 to JP1, L2 to L1, LDO2 to LDO1, SD2 to SD1, USB2 to USB1
Connections:
- net !CTS: now also U2.!CTS; no longer U5.!CTS
- net 3.3V: now also C14.2, C2.2, C20.2, C21.1, C9.1, D3.C, J2.4, LED3.A, LED4.A, R10.2, U1.VDD, U2.!RESET, U2.VCCIO, U4.VBAT; no longer C12.2, C17.2, C2.1, C25.1, C5.2, D1.C, LED5.A, LED6.A, R17.2, R5.2, U2.VDD, U3.VBAT, U5.!RESET, U5.VCCIO
- net A4/BATT: now also R8.1, R9.2, U1.P0.28/AIN4; no longer R15.1, R16.2, U2.P0.28/AIN4
- net A6/TIA: now also J2.6, U1.P0.30/AIN6; no longer U2.P0.30/AIN6
- net A7/PPG: now also J2.7, U1.P0.31/AIN7; no longer U2.P0.31/AIN7
- net D11/SW1: now also SW3.1, U1.P0.11; no longer SW1.1, U2.P0.11
- net D15/SW2: now also SW4.1, U1.P0.15; no longer SW2.1, U2.P0.15
- net D16/CS.OLED: now also U1.P0.16, U4./CS; no longer U2.P0.16, U3./CS
- net D27/CHRG.STATUS: now also R3.1, U1.P0.27; no longer R14.1, U2.P0.27
- net D29/LED.CTRL: now also J2.5, U1.P0.29/AIN5; no longer U2.P0.29/AIN5
- net D3/RESET.OLED: now also U1.P0.03/AIN1, U4./RES; no longer U2.P0.03/AIN1, U3./RES
- net D4/DC.OLED: now also U1.P0.04/AIN2, U4.DC/I2C_SA0; no longer U2.P0.04/AIN2, U3.DC/I2C_SA0
- net D5/CD1: now also U1.P0.05/AIN3; no longer U2.P0.05/AIN3
- net D7/SD.CS: now also U1.P0.07; no longer U2.P0.07
- net DFU: now also SW1.B, U1.P0.20; no longer SW3.B, U2.P0.20
- net DTR: now also C12.1, U2.!DTR; no longer C14.1, U5.!DTR
- net FRST: now also U1.P0.22; no longer U2.P0.22
- net FT3V3: now also U2.3V3OUT; no longer U5.3V3OUT
- net GND: now also C1.2, C11.1, C13.2, C14.1, C15.1, C2.1, C21.2, C4.2, C7.1, J1.1, J2.3, LED1.C, LED2.C, R16.2, R5.1, R9.1, SW1.A, SW2.B, SW3.3, SW4.3, U1.GND@1, U1.GND@2, U1.GND@3, U1.GND@4, U2.GND@16, U2.GND@6, U4.BS0, U4.BS2, U4.NC(GND)@1, U4.NC(GND)@2, U4.VLSS; no longer C11.2, C12.1, C16.1, C18.1, C2.2, C24.1, C25.2, C26.2, C27.1, C6.2, C7.2, J2.1, LED3.C, LED4.C, R16.1, R17.1, R6.1, R7.2, SW1.3, SW1.4, SW2.3, SW2.4, SW3.A, SW4.B, U2.GND@1, U2.GND@2, U2.GND@3, U2.GND@4, U3.BS0, U3.BS2, U3.NC(GND)@1, U3.NC(GND)@2, U3.VLSS, U5.GND@16, U5.GND@6
- net LED1: now also R4.2, U1.P0.17; no longer R3.2, U2.P0.17
- net LED2: now also R7.2, U1.P0.19; no longer R4.2, U2.P0.19
- net MISO: now also U1.P0.14; no longer U2.P0.14
- net MOSI: now also U1.P0.13, U4.D1/SPI_SDIN/I2C_SDA; no longer U2.P0.13, U3.D1/SPI_SDIN/I2C_SDA
- net N$1: now also R13.2, U4.BS1; no longer R6.2, U3.BS1
- net N$10: now also LED2.A, R7.1; no longer LED4.A, R4.1
- net N$11: now also U1.DCC; no longer U2.DCC
- net N$12: now also C1.1, U1.DEC4; no longer C7.1, U2.DEC4
- net N$13: now also C15.2, U4.VCC; no longer C16.2, U3.VCC
- net N$15: now also C17.2, U4.VCOMH; no longer C18.2, U3.VCOMH
- net N$17: now also R5.2; no longer R13.2
- net N$19: now also U3.OSCO, XTAL2.1; no longer U4.OSCO, XTAL3.1
- net N$2: now also R16.1, U4.IREF; no longer R7.1, U3.IREF
- net N$20: now also U3.OSCI, XTAL2.2; no longer U4.OSCI, XTAL3.2
- net N$23: now also R11.2, U2.USBDM; no longer R12.2, U5.USBDM
- net N$24: now also R12.2, U2.USBDP; no longer R18.2, U5.USBDP
- net N$25: now also LED3.C, R14.2; no longer LED5.C, R19.2
- net N$26: now also LED4.C, R15.2; no longer LED6.C, R20.2
- net N$3: now also C18.2, U4.C2P; no longer C13.2, U3.C2P
- net N$4: now also U1.P0.00/XL1, XTAL1.1; no longer U2.P0.00/XL1, XTAL2.1
- net N$5: now also C18.1, U4.C2N; no longer C13.1, U3.C2N
- net N$6: now also C4.1, U1.P0.01/XL2, XTAL1.2; no longer C9.1, U2.P0.01/XL2, XTAL2.2
- net N$7: now also C16.2, U4.C1P; no longer C15.2, U3.C1P
- net N$8: now also C16.1, U4.C1N; no longer C15.1, U3.C1N
- net N$9: now also LED1.A, R4.1; no longer LED3.A, R3.1
- net P0.09/NFC1: now also U1.P0.09; no longer C11.1, U2.P0.09
- net P0.10/NFC2: now also U1.P0.10; no longer C10.1, U2.P0.10
- net RESET: now also C12.2, D3.A, R10.1, SW2.A, U1.P0.21/RESET; no longer C14.2, D1.A, R5.1, SW4.A, U2.P0.21/RESET
- net RXD.FT: now also R18.1, U2.RXD; no longer R22.1, U5.RXD
- net RXD.NRF: now also R17.2, U1.P0.08; no longer R21.2, U2.P0.08
- net RXLED: now also R14.1, U2.CBUS1; no longer R19.1, U5.CBUS1
- net SCK: now also U1.P0.12, U4.D0/SPI_SCLK/I2C_SCK; no longer U2.P0.12, U3.D0/SPI_SCLK/I2C_SCK
- net SCL: now also J2.2, U1.P0.26, U3.SCL; no longer U2.P0.26, U4.SCL
- net SDA: now also J2.1, U1.P0.25, U3.SDA; no longer U2.P0.25, U4.SDA
- net SWCLK: now also U1.SWDCLK; no longer U2.SWDCLK
- net SWDIO: now also U1.SWDIO; no longer U2.SWDIO
- net SWO: now also U1.P0.18/SWO; no longer U2.P0.18/SWO
- net TXD.FT: now also R17.1, U2.TXD; no longer R21.1, U5.TXD
- net TXD.NRF: now also R18.2, U1.P0.06; no longer R22.2, U2.P0.06
- net TXLED: now also R15.1, U2.CBUS2; no longer R20.1, U5.CBUS2
- net USB+: now also C13.1, R12.1; no longer C6.1, R18.1
- net USB-: now also C11.2, R11.1; no longer C20.2, R12.1
- net VBATT: now also U3.VBAT; no longer U4.VBAT
- net VIN: now also C5.2, C7.2, D1.C, R3.2; no longer C24.2, C27.2, D4.C, R14.2
- net VLIPO: now also C10.1, D1.A, J1.2, R8.2; no longer C26.1, D4.A, J2.2, R15.2
- net V_USB: now also U2.VCC; no longer U5.VCC
Other:
- note added: "Connection to lower board"
- note added: "Cortex Debugger/ Programmer"
- note added: "I2C Address: 0x2C"
- note removed: "Cortex Debugger/Programmer"
- moved on the sheet: C10, C11, C12, C13, C14, C15, C16, C17, C18, C2, C20, C5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

Commit message: take7
Parts:
- removed C10, C5: 4.7u, LinnesLab-Passives:CAPACITOR0603
- removed C21, C7, C9: 1u, LinnesLab-Passives:CAPACITOR0603
- removed CHRG1: MCP73831, LinnesLab-Power:MCP73831
- removed LDO1: MIC5504, LinnesLab-Power:MIC5504
- removed R3: 100k, LinnesLab-Passives:RESISTOR0603
- removed R5: (no value), LinnesLab-Passives:RESISTOR0603
- removed SD1: (no value), LinnesLab-Connectors:MICROSD
- removed U3: PCF8523, LinnesLab-Clocks:PCF8523
- removed XTAL2: 32.7680kHz, LinnesLab-Clocks:CRYSTALECS-.327-12.5-12-C-TR
- C17: device LinnesLab-Passives:CAPACITOR0402 -> LinnesLab-Passives:CAPACITOR0603
Connections:
- removed net A4/BATT: R8.1, R9.2, U1.P0.28/AIN4
- removed net A6/TIA: J2.6, U1.P0.30/AIN6
- removed net A7/PPG: J2.7, U1.P0.31/AIN7
- removed net CD2: SD1.CARD_DETECT1
- removed net D29/LED.CTRL: J2.5, U1.P0.29/AIN5
- removed net N$17: CHRG1.PROG, R5.2
- removed net N$19: U3.OSCO, XTAL2.1
- removed net N$20: U3.OSCI, XTAL2.2
- removed net VBATT: U3.VBAT
- new net A4/PPG: J2.7, U1.P0.28/AIN4
- new net A5/TIA: J2.6, U1.P0.29/AIN5
- new net A7/BATT: R8.1, R9.2, U1.P0.31/AIN7
- new net D30/LED.CTRL: J2.5, U1.P0.30/AIN6
- net 3.3V: no longer C21.1, C9.1, LDO1.OUT, SD1.VDD, U3.VDD
- net D27/CHRG.STATUS: no longer CHRG1.STAT, R3.1
- net D5/CD1: no longer SD1.CARD_DETECT
- net D7/SD.CS: no longer SD1.CS
- net GND: no longer C10.2, C21.2, C5.1, C7.1, C9.2, CHRG1.VSS, LDO1.GND, R5.1, SD1.GND, SD1.GND1, SD1.VSS, U3.VSS
- net MISO: no longer SD1.DATA_OUT
- net MOSI: no longer SD1.DATA_IN
- net SCK: no longer SD1.SCLK
- net SCL: no longer U3.SCL
- net SDA: no longer U3.SDA
- net VIN: no longer C5.2, C7.2, CHRG1.VIN, LDO1.EN, LDO1.IN, R3.2
- net VLIPO: no longer C10.1, CHRG1.VBAT
Other:
- note removed: "Back-up battery if desired"
- note removed: "Connect MISO, MOSI, and SCK to appropriate pins on microcontroller. Those are SPI pins and are generally prespecified. You have more flexibility with the SD.CS pin."
- note removed: "Digital Output"
- note removed: "I2C Address = 0x68h"
- note removed: "Real-Time Clock"
- note removed: "SD Card"

Commit message: take 8
Parts:
- added C5, C6: 4.7u, LinnesLab-Passives:CAPACITOR0603
- added C7, C9: 1u, LinnesLab-Passives:CAPACITOR0603
- added CHRG1: MCP73831, LinnesLab-Power:MCP73831
- added LDO1: MIC5504, LinnesLab-Power:MIC5504
- added R3: 100k, LinnesLab-Passives:RESISTOR0603
- added R5: (no value), LinnesLab-Passives:RESISTOR0603
Connections:
- new net N$16: CHRG1.PROG, R5.2
- net 3.3V: now also C9.1, LDO1.OUT
- net D27/CHRG.STATUS: now also CHRG1.STAT, R3.1
- net GND: now also C5.2, C6.1, C7.1, C9.2, CHRG1.VSS, LDO1.GND, R5.1
- net VIN: now also C6.2, C7.2, CHRG1.VIN, LDO1.EN, LDO1.IN, R3.2
- net VLIPO: now also C5.1, CHRG1.VBAT
Other:
- note added: "Digital Output"

Commit message: 'take8'
Parts:
- removed C19, C20: 2.2uF, LinnesLab-Passives:CAPACITOR0402
- removed R18: 0, LinnesLab-Passives:RESISTOR0603
- removed U4: (no value), LinnesLab-Displays:DISP_OLED_UG-2864HSWEG01-NO-WRAPAROUND
- added C10: 2.2uF, LinnesLab-Passives:CAPACITOR0402
- added C8: 4.7u, LinnesLab-Passives:CAPACITOR0603
- added R6: 1k, LinnesLab-Passives:RESISTOR0603
- added U3: FT231XS, LinnesLab-DigitalIC:FT231XS
- C11: value 47p -> 2.2uF
- C12, C14: value 100n -> 2.2uF; device LinnesLab-Passives:CAPACITOR0603 -> LinnesLab-Passives:CAPACITOR0402
- C13: value 47p -> 2.2uF; device LinnesLab-Passives:CAPACITOR0603 -> LinnesLab-Passives:CAPACITOR0402
- C15: value 10uF -> 47p
- C16: value 2.2uF -> 47p; device LinnesLab-Passives:CAPACITOR0402 -> LinnesLab-Passives:CAPACITOR0603
- C17: value 2.2uF -> 100n
- C18: value 2.2uF -> 100n; device LinnesLab-Passives:CAPACITOR0402 -> LinnesLab-Passives:CAPACITOR0603
- C6: value 4.7u -> 1u
- C9: value 1u -> 10uF
- R10: value 10k -> 390k
- R13: value 10k -> 1k
- R15: value 1k -> 0
- R16: value 390k -> 0
- R17: value 0 -> 10k
- R7: value 1k -> 100k
- R9: value 100k -> 10k
- SW2: value (none) -> SWITCH.MOM; device LinnesLab-Switches:SPST-PTS830GG140-COPY.1-3 -> LinnesLab-Switches:SWITCH.MOM
- SW4: value SWITCH.MOM -> (none); device LinnesLab-Switches:SWITCH.MOM -> LinnesLab-Switches:SPST-PTS830GG140-COPY.1-3
- U2: value FT231XS -> (none); device LinnesLab-DigitalIC:FT231XS -> LinnesLab-Displays:DISP_OLED_UG-2864HSWEG01-NO-WRAPAROUND
Connections:
- net !CTS: now also U3.!CTS; no longer U2.!CTS
- net 3.3V: now also C13.2, C17.2, C7.1, R17.2, U2.VBAT, U2.VDD, U3.!RESET, U3.VCCIO; no longer C19.2, C20.2, C9.1, R10.2, U2.!RESET, U2.VCCIO, U4.VBAT, U4.VDD
- net A7/BATT: now also R7.1, R8.2; no longer R8.1, R9.2
- net D11/SW1: now also SW2.1; no longer SW3.1
- net D15/SW2: now also SW3.1; no longer SW4.1
- net D16/CS.OLED: now also U2./CS; no longer U4./CS
- net D3/RESET.OLED: now also U2./RES; no longer U4./RES
- net D4/DC.OLED: now also U2.DC/I2C_SA0; no longer U4.DC/I2C_SA0
- net DTR: now also C18.1, U3.!DTR; no longer C12.1, U2.!DTR
- net FT3V3: now also U3.3V3OUT; no longer U2.3V3OUT
- net GND: now also C13.1, C16.2, C5.1, C7.2, C8.2, C9.1, R10.2, R8.1, SW2.3, SW4.B, U2.BS0, U2.BS2, U2.NC(GND)@1, U2.NC(GND)@2, U2.VLSS, U2.VSS, U3.GND@16, U3.GND@6; no longer C13.2, C19.1, C20.1, C5.2, C7.1, C9.2, R13.1, R16.2, SW2.B, SW4.3, U2.GND@16, U2.GND@6, U4.BS0, U4.BS2, U4.NC(GND)@1, U4.NC(GND)@2, U4.VLSS, U4.VSS
- net LED2: now also R6.2; no longer R7.2
- net MOSI: now also U2.D1/SPI_SDIN/I2C_SDA; no longer U4.D1/SPI_SDIN/I2C_SDA
- net N$1: now also R9.2, U2.BS1; no longer R13.2, U4.BS1
- net N$10: now also R6.1; no longer R7.1
- net N$13: now also C9.2, U2.VCC; no longer C15.2, U4.VCC
- net N$15: now also C11.2, U2.VCOMH; no longer C17.2, U4.VCOMH
- net N$2: now also R10.1, U2.IREF; no longer R16.1, U4.IREF
- net N$23: now also U3.USBDM; no longer U2.USBDM
- net N$24: now also U3.USBDP; no longer U2.USBDP
- net N$25: now also R13.2; no longer R14.2
- net N$26: now also R14.2; no longer R15.2
- net N$3: now also C12.2, U2.C2P; no longer C18.2, U4.C2P
- net N$5: now also C12.1, U2.C2N; no longer C18.1, U4.C2N
- net N$7: now also C10.2, U2.C1P; no longer C16.2, U4.C1P
- net N$8: now also C10.1, U2.C1N; no longer C16.1, U4.C1N
- net RESET: now also C18.2, R17.1, SW4.A; no longer C12.2, R10.1, SW2.A
- net RXD.FT: now also R16.1, U3.RXD; no longer R18.1, U2.RXD
- net RXD.NRF: now also R15.2; no longer R17.2
- net RXLED: now also R13.1, U3.CBUS1; no longer R14.1, U2.CBUS1
- net SCK: now also U2.D0/SPI_SCLK/I2C_SCK; no longer U4.D0/SPI_SCLK/I2C_SCK
- net TXD.FT: now also R15.1, U3.TXD; no longer R17.1, U2.TXD
- net TXD.NRF: now also R16.2; no longer R18.2
- net TXLED: now also R14.1, U3.CBUS2; no longer R15.1, U2.CBUS2
- net USB+: now also C16.1; no longer C13.1
- net USB-: now also C15.2; no longer C11.2
- net VIN: now also C5.2; no longer C7.2
- net VLIPO: now also C8.1, R7.2; no longer C5.1, R8.2
- net V_USB: now also U3.VCC; no longer U2.VCC
Other:
- note added: "0 Phm Resistors in case I mixed up TX/RX"
- note added: "AAlsaati - SmartWatch v1 MAR 20, 2021"
- note added: "Connection Headers from Top to bottom"
- note added: "Diodes Switch from LiPo power to USB when USB is connected the USB powers then charges battery"
- note added: "R5 set charge current i_charge = 1000V/R5 per MCP73831 Datasheet"
- note added: "Voltage Divider used to monitor battery voltage"
- moved on the sheet: C11, C12, C13, C14, C15, C16, C17, C18, C5, C6, C7, C9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
